File: hardware/pocket-pet/pocket-pet.kicad_sch (KiCad schematic)
At the start: 0 parts

Commit message: Power tree: USB-C, MCP73831 charger, battery, switch, custom SS12D00G3 footprint
Parts:
- added C1, C2: 4.7uF, Capacitor_SMD:C_0805_2012Metric_Pad1.18x1.45mm_HandSolder, symbol Device:C
- added J1: USB_C_Receptacle_USB2.0_16P, Connector_USB:USB_C_Receptacle_HRO_TYPE-C-31-M-12, symbol Connector:USB_C_Receptacle_USB2.0_16P
- added J2: Conn_01x02, Connector_JST:JST_PH_S2B-PH-K_1x02_P2.00mm_Horizontal, symbol Connector_Generic:Conn_01x02
- added R1, R2, R3: 5.1k, Resistor_SMD:R_0805_2012Metric_Pad1.20x1.40mm_HandSolder, symbol Device:R
- added SW1: SW_SPDT, pocket-pet:SW_Slide_SS12D00G3_P2.5mm, symbol Switch:SW_SPDT
- added U1: MCP73831-2-OT, Package_TO_SOT_SMD:SOT-23-5, symbol Battery_Management:MCP73831-2-OT
Connections:
- new net: R1.2, U1.5 (PROG)
- new net: J1.A5 (CC1), R2.1
- new net: J1.B5 (CC2), R3.1
- new net GND: C1.2, C2.2, J1.A1 (GND), J1.A12 (GND), J1.B1 (GND), J1.B12 (GND), J1.SH (SHIELD), J2.2 (Pin_2), R1.1, R2.2, R3.2, U1.2 (V_{SS})
- new net VBAT: C2.1, J2.1 (Pin_1), SW1.2 (B), U1.3 (V_{BAT})
- new net VBAT_SW: SW1.1 (A)
- new net VBUS: C1.1, J1.A4 (VBUS), J1.A9 (VBUS), J1.B4 (VBUS), J1.B9 (VBUS), U1.4 (V_{DD})

Commit message: MCU: power pins, decoupling, BOOT0 pulldown, NRST cap
Parts:
- added C10: 4.7uF, Capacitor_SMD:C_0805_2012Metric_Pad1.18x1.45mm_HandSolder, symbol Device:C
- added C11, C5, C6, C7, C8, C9: 100nF, Capacitor_SMD:C_0805_2012Metric_Pad1.18x1.45mm_HandSolder, symbol Device:C
- added C3: 1uF, Capacitor_SMD:C_0805_2012Metric_Pad1.18x1.45mm_HandSolder, symbol Device:C
- added C4: 2.2uF, Capacitor_SMD:C_0805_2012Metric_Pad1.18x1.45mm_HandSolder, symbol Device:C
- added R4: 10k, Resistor_SMD:R_0805_2012Metric_Pad1.20x1.40mm_HandSolder, symbol Device:R
- added TP1: TestPoint, TestPoint:TestPoint_Pad_D1.5mm, symbol Connector:TestPoint
- added U2: MCP1700x-330xxTT, Package_TO_SOT_SMD:SOT-23, symbol Regulator_Linear:MCP1700x-330xxTT
- added U3: STM32L433CCTx, Package_QFP:LQFP-48_7x7mm_P0.5mm, symbol MCU_ST_STM32L4:STM32L433CCTx
Connections:
- net GND: now also C10.2, C11.2, C3.2, C4.2, C5.2, C6.2, C7.2, C8.2, C9.2, R4.2, U2.1 (GND), U3.23 (VSS), U3.35 (VSS), U3.47 (VSS), U3.8 (VSSA)
- net VBAT_SW: now also C3.1, U2.3 (VI)
- new net: R4.1, U3.44 (PH3)
- new net: C11.1, U3.7 (NRST)
- new net 3V3: C10.1, C4.1, C5.1, C6.1, C7.1, C8.1, C9.1, TP1.1, U2.2 (VO), U3.1 (VBAT), U3.24 (VDD), U3.36 (VDDUSB), U3.48 (VDD), U3.9 (VDDA)

Commit message: Schematic complete: display, accelerometer, buttons, ERC clean
Parts:
- added J3: Conn_01x06, Connector_PinHeader_2.54mm:PinHeader_1x06_P2.54mm_Vertical, symbol Connector_Generic:Conn_01x06
- added J4: Conn_01x07, Connector_PinHeader_2.54mm:PinHeader_1x07_P2.54mm_Vertical, symbol Connector_Generic:Conn_01x07
- added J5: Conn_01x08, Connector_PinHeader_2.54mm:PinHeader_1x08_P2.54mm_Vertical, symbol Connector_Generic:Conn_01x08
- added R5, R6: 0R, Resistor_SMD:R_0805_2012Metric_Pad1.20x1.40mm_HandSolder, symbol Device:R
- added R7, R8: 4.7k, Resistor_SMD:R_0805_2012Metric_Pad1.20x1.40mm_HandSolder, symbol Device:R
- added SW2, SW3: SW_Push, Button_Switch_THT:SW_PUSH_6mm, symbol Switch:SW_Push
Connections:
- net 3V3: now also J3.1 (Pin_1), J5.6 (Pin_6), R5.1, R6.2, R7.2, R8.2
- net GND: now also J3.6 (Pin_6), J4.1 (Pin_1), J5.2 (Pin_2), J5.5 (Pin_5), SW2.2, SW3.2
- net BTN_A: now reaches U3.10 (PA0)
- net BTN_A: now also SW2.1
- net BTN_B: now reaches U3.11 (PA1)
- net BTN_B: now also SW3.1
- net OLED_CS: now reaches U3.14 (PA4)
- net OLED_CS: now also J4.7 (Pin_7)
- net at U3.15 (PA5): now also J4.3 (Pin_3)
- net at U3.17 (PA7): now also J4.4 (Pin_4)
- net OLED_DC: now reaches U3.18 (PB0)
- net OLED_DC: now also J4.6 (Pin_6)
- net OLED_RST: now reaches U3.19 (PB1)
- net OLED_RST: now also J4.5 (Pin_5)
- net SWDIO: now reaches U3.34 (PA13)
- net SWDIO: now also J3.2 (Pin_2)
- net SWCLK: now reaches U3.37 (PA14)
- net SWCLK: now also J3.3 (Pin_3)
- net SWO: now reaches U3.39 (PB3)
- net SWO: now also J3.4 (Pin_4)
- net ACCEL_INT1: now reaches U3.41 (PB5)
- net ACCEL_INT1: now also J5.8 (Pin_8)
- net ACCEL_SCL: now reaches U3.42 (PB6)
- net ACCEL_SCL: now also J5.3 (Pin_3), R7.1
- net ACCEL_SDA: now reaches U3.43 (PB7)
- net ACCEL_SDA: now also J5.4 (Pin_4), R8.1
- net NRST: now reaches C11.1, U3.7 (NRST)
- net NRST: now also J3.5 (Pin_5)
- new net: J4.2 (Pin_2), R5.2
- new net: J5.1 (Pin_1), R6.1
Other:
- moved on the sheet: C1, C2, C3, C4, J1, J2, R1, R2, R3, SW1, TP1, U1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

Commit message: Layout complete, DRC clean, boards ordered
Parts:
- removed J5: Conn_01x08, Connector_PinHeader_2.54mm:PinHeader_1x08_P2.54mm_Vertical, symbol Connector_Generic:Conn_01x08
- added J6: Conn_01x11, Connector_PinHeader_2.54mm:PinHeader_1x11_P2.54mm_Vertical, symbol Connector_Generic:Conn_01x11
- added TP2: TestPoint, TestPoint:TestPoint_THTPad_D2.0mm_Drill1.0mm, symbol Connector:TestPoint
Connections:
- net 3V3: now also J6.6 (Pin_6)
- net ACCEL_INT1: now also J6.7 (Pin_7)
- net ACCEL_SCL: now also J6.3 (Pin_3)
- net ACCEL_SDA: now also J6.4 (Pin_4)
- net GND: now also J6.2 (Pin_2), J6.5 (Pin_5), TP2.1
- net at R6.1: now also J6.1 (Pin_1)
- no-connect marks 0 -> 36
Other:
- moved on the sheet: R4, R6
